File: output/pcbs/right.kicad_pcb (KiCad board)
At the start: 2 copper layers, 116.5 x 114 mm, 63 parts

Commit message: right side is alsmost finished
Parts:
- moved S1 244.7 mm to (209.5, 126.5)
- moved S2 244.7 mm to (209.5, 107.5)
- moved S3 244.7 mm to (209.5, 88.5)
- moved S4 244.7 mm to (209.5, 69.5)
- moved S5 244.7 mm to (209.5, 50.5)
- moved D3 231.9 mm to (198.5, 96.0)
- moved D4 231.0 mm to (198.5, 77.0)
- moved D1 230.0 mm to (198.5, 130.5)
- moved D2 229.6 mm to (198.5, 115.0)
- moved D5 228.9 mm to (198.0, 57.5)
- moved S10 211.8 mm to (188.8, 50.5)
- moved S6 211.8 mm to (188.8, 126.5)
- moved S7 211.8 mm to (188.8, 107.5)
- moved S8 211.8 mm to (188.8, 88.5)
- moved S9 211.8 mm to (188.8, 69.5)
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Routing:
- net P115: track 211.6 -> 339.1 mm
- net P017: track 141.8 -> 76.8 mm
- net P002: track 186.8 -> 250.5 mm
- net RAW: track 31.2 -> 69.3 mm, vias 0 -> 2
- net P113: track 297.5 -> 260.8 mm
- net P011: track 133.5 -> 99.1 mm
- net inner_bottom: track 32.8 -> 7.46 mm
- net inner_num: track 32.5 -> 7.78 mm
- net P100: track 134.9 -> 110.8 mm
- net index_home: track 31.2 -> 7.20 mm
- net index_top: track 30.6 -> 7.20 mm
- net index_bottom: track 29.7 -> 7.20 mm
- net outer_home: track 28.1 -> 7.04 mm
- net middle_num: track 28.3 -> 7.66 mm
- net ring_top: track 27.6 -> 7.04 mm
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Other:
- board size 116.5 x 114 mm -> 118.4 x 114.2 mm
